Commit message: Update base_link

File: raspitank_description/urdf/camera.xacro (robot description, xacro)
@@ -13,5 +13,5 @@
   <joint name="camera_joint" type="fixed">
     <origin xyz="0.075198 -0.00075 0.088" rpy="0 0 0"/>
-    <parent link="chassis_link"/>
+    <parent link="base_link"/>
     <child link="camera_link"/>
   </joint>

File: raspitank_description/urdf/gazebo_control.xacro (robot description, xacro)
@@ -11,5 +11,5 @@
       <wheelSeparation>0.2</wheelSeparation>
       <wheelDiameter>0.06</wheelDiameter>
-      <robotBaseFrame>base_link</robotBaseFrame>
+      <robotBaseFrame>base_footprint</robotBaseFrame>
       <torque>20</torque>
       <topicName>cmd_vel</topicName>

File: raspitank_description/urdf/lidar.xacro (robot description, xacro)
@@ -21,5 +21,5 @@
     <joint name="lidar_joint" type="fixed">
         <origin xyz="0.004 0.0 0.122" rpy="0 0 ${pi}"/>
-        <parent link="chassis_link"/>
+        <parent link="base_link"/>
         <child link="lidar_link"/>
     </joint>

File: raspitank_description/urdf/raspitank_core.xacro (robot description, xacro)
@@ -13,21 +13,12 @@
   <!-- Distance between centre of wheel and robot base -->
   <xacro:property name="wheel_zoff" value="0.01"/>
-  <!-- BASE LINK -->
-  <link name="base_link">
-  </link>
   <!-- BASE_FOOTPRINT LINK -->
-  <joint name="base_footprint_joint" type="fixed">
-    <parent link="base_link"/>
-    <child link="base_footprint"/>
-    <origin xyz="0 0 0" rpy="0 0 0"/>
-  </joint>
-  <link name="base_footprint">
-  </link>
+  <link name="base_footprint"/>
   <!-- CHASSIS LINK -->
-<joint name="chassis_joint" type="fixed">
-  <parent link="base_link"/>
-  <child link="chassis_link"/>
+<joint name="base_joint" type="fixed">
+  <parent link="base_footprint"/>
+  <child link="base_link"/>
 </joint>
-<link name="chassis_link">
+<link name="base_link">
   <visual>
     <origin xyz="0 0 0" rpy="0 0 0"/>
@@ -47,10 +38,10 @@
     </xacro:box_inertia>
 </link>
-<gazebo reference="chassis_link">
+<gazebo reference="base_link">
     <material>Gazebo/White</material>
 </gazebo>
 <!-- LEFT BACK WHEEL -->
 <!-- <joint name="left_wheel_joint" type="continuous">
-  <parent link="chassis_link"/>
+  <parent link="base_link"/>
   <child link="left_wheel"/>
   <origin xyz="-0.112746 0.07275 0.053" rpy="0 0 0"/>
@@ -58,5 +49,5 @@
 </joint> -->
 <joint name="left_wheel_joint" type="continuous">
-  <parent link="chassis_link"/>
+  <parent link="base_link"/>
   <child link="left_wheel"/>
   <origin xyz="0.01 0.1 0.03" rpy="0 0 0"/>
@@ -87,5 +78,5 @@
 <!-- RIGHT BACK WHEEL -->
 <!-- <joint name="right_wheel_joint" type="continuous">
-  <parent link="chassis_link"/>
+  <parent link="base_link"/>
   <child link="right_wheel"/>
   <origin xyz="-0.112746 -0.07225 0.053" rpy="0 0 0"/>
@@ -93,5 +84,5 @@
 </joint> -->
 <joint name="right_wheel_joint" type="continuous">
-  <parent link="chassis_link"/>
+  <parent link="base_link"/>
   <child link="right_wheel"/>
   <origin xyz="0.01 -0.1 0.03" rpy="0 0 0"/>
@@ -132,5 +123,5 @@
   </link>
   <joint name="caster_wheel_joint" type="fixed">
-    <parent link="chassis_link"/>
+    <parent link="base_link"/>
     <child link="caster_wheel"/>
     <origin xyz="0.096 0 0" rpy="0 0 0"/>
