Commit message: Update README.md

File: raspitank_description/urdf/lidar.xacro (robot description, xacro)
@@ -1,4 +1,9 @@
 <?xml version="1.0" ?>
 <robot xmlns:xacro="http://ros.org/wiki/xacro">raspitank_description
+    <joint name="lidar_joint" type="fixed">
+        <origin xyz="0.004 0.0 0.122" rpy="0 0 ${pi}"/>
+        <parent link="base_link"/>
+        <child link="lidar_link"/>
+    </joint>
     <link name="lidar_link">
         <visual>
@@ -19,9 +24,4 @@
         </xacro:cylinder_inertia>
     </link>
-    <joint name="lidar_joint" type="fixed">
-        <origin xyz="0.004 0.0 0.122" rpy="0 0 ${pi}"/>
-        <parent link="base_link"/>
-        <child link="lidar_link"/>
-    </joint>
     <gazebo reference="lidar_link">
         <material>Gazebo/Blue</material>

File: raspitank_description/urdf/ros2_control.xacro (robot description, xacro)
@@ -12,5 +12,5 @@
             <param name="baud_rate">57600</param>
             <param name="timeout_ms">1000</param>
-            <param name="enc_counts_per_rev">3436</param>
+            <param name="enc_counts_per_rev">1436</param>
             <param name="pid_p">20</param>
             <param name="pid_d">12</param>
